File: Hardware/Retrospector_Components.kicad_pcb (KiCad board)
At the start: 4 copper layers, 60 x 110 mm, 123 parts, among them J1 SWD_Header, J2 Eurorack_10_pin_power, J3 Conn_01x08_Male, J4 Conn_01x08_Male, J5 Conn_01x08_Male, J6 Conn_01x08_Male, J7 USB_B_Micro, U1 STM32H743ZITx, U2 IS42S16400J-xC, U3 PCM5100APW, U4 SSI2164, U5 MCP6004, U6 MCP6004, U7 TL074, U8 LM1117-3.3, Y1 8MHz 20pF

Commit message: Started adding LCD support
Connections:
- net /FMC_SD~E1 renamed /FMC_SD~{E1}
- net /FMC_SD~WE renamed /FMC_SD~{WE}
- net /FMC_~BL0 renamed /FMC_~{BL0}
- net /FMC_~BL1 renamed /FMC_~{BL1}
- net /FMC_~CAS renamed /FMC_~{CAS}
- net /FMC_~RAS renamed /FMC_~{RAS}
Routing:
- added copper zone on In2.Cu, net +3.3VA
- added copper zone on In2.Cu, net +3V3
- added copper zone on In1.Cu, net GND
- removed copper zone on Power.Rails, net +3.3VA
- removed copper zone on Power.Rails, net +3V3
- removed copper zone on Ground.Fill, net GND
Other:
- net class Default removed
- net class Wide_Power removed
