File: Hardware/Retrospector_Components.kicad_sch (KiCad schematic)
At the start: 123 parts, among them J1 SWD_Header, J2 Eurorack_10_pin_power, J3 Conn_01x08_Male, J4 Conn_01x08_Male, J5 Conn_01x08_Male, J6 Conn_01x08_Male, J7 USB_B_Micro, U1 STM32H743ZITx, U2 IS42S16400J-xC, U3 PCM5100APW, U4 SSI2164, U5 MCP6004, U6 MCP6004, U7 TL074, U8 LM1117-3.3, Y1 8MHz 20pF

Commit message: Performance testing updates
Other:
- note added: "PC10 SPI3_CLK (was LED1) PC11 DC (was LED2) PC12 SPI3_MOSI (was DELAY_CHORUS) PE2 - debug (was MODE1) PE3 - debug (was MODE2)"
