File: Hardware/Combined_Controls_Components/Kishoof_Components.kicad_sch (KiCad schematic)
At the start: 98 parts, among them J1 Conn_01x12_Pin, J2 Conn_01x12_Pin, J3 Conn_01x12_Pin, J4 Conn_01x12_Pin, J5 Eurorack_10_pin_power, J6 SWD_Header, J7 Conn_01x02_Pin, U1 STM32H7B0VBTx, U2 PCM5100APW, U3 TPS561201, U4 LT1117-3.3, U5 MCP6002, U6 MX25LM51245G, U7 MCP6004, U8 TL072, Y1 8MHz 20pF

Commit message: Separated PCB controls and components
Parts:
- removed J1, J2, J3, J4: Conn_01x12_Pin, Connector_PinHeader_2.54mm:PinHeader_1x12_P2.54mm_Vertical, symbol Connector:Conn_01x12_Pin
- removed J7: Conn_01x02_Pin, Connector_PinHeader_2.54mm:PinHeader_1x02_P2.54mm_Vertical, symbol Connector:Conn_01x02_Pin
- added JP1: Jumper, Jumper:SolderJumper-2_P1.3mm_Open_RoundedPad1.0x1.5mm, symbol Jumper:Jumper_2_Open
- added U9: STF202-22T1G, Custom_Footprints:STF202-22T1G, symbol STF202-22T1G:STF202-22T1G
- renumbered J6 to J1, J5 to J2
Connections:
- net B_Octave_Btn: now also U1.56 (PD9); no longer U1.57 (PD10)
- net ChB_Mix: now also U1.42 (PE12); no longer U1.55 (PD8)
- net ChB_RM: now also U1.43 (PE13); no longer U1.56 (PD9)
- net Encoder_Btn: now also U1.88 (PD7); no longer U1.3 (PE4)
- net GND: now also U9.6 (GND)
- net USB_DM: now also U9.2 (D1_OUT)
- net USB_DP: now also U9.3 (D2_OUT)
- net USB_VBUS: now also JP1.2 (B)
- net WavetablePosA_CV: now also U1.35 (PB1); no longer U1.31 (PA7)
- net Wavetable_Pos_A_Pot: now also U1.31 (PA7); no longer U1.35 (PB1)
- new net: JP1.1 (A), U9.1 (VBUS)
- new net USB_D+: U9.4 (D2_IN)
- new net USB_D-: U9.5 (D1_IN)
Other:
- added sheet Kishoof_Controls (Kishoof_Controls.kicad_sch)
